Commit message: solved controllers errors

File: description/robot_core.xacro (robot description, xacro)
@@ -40,5 +40,5 @@
         <child link="link_1" />
         <limit lower="0" upper="${2*pi}" velocity="${joint_1_velocity}" effort="${joint_1_effort}" />
-        <dynamics damping="1.0" friction="1.0"/>
+        <!-- <dynamics damping="1.0" friction="1.0"/> -->
     </joint>
     <!-- link_1 describes the link_1 of the arm -->
@@ -73,5 +73,5 @@
         <child link="link_2" />
         <limit lower="0" upper="${2*pi}" velocity="${joint_2_velocity}" effort="${joint_2_effort}" />
-        <dynamics damping="1.0" friction="1.0"/>
+        <!-- <dynamics damping="1.0" friction="1.0"/> -->
     </joint>
     <!-- link_2 describes the link_2 of the arm -->

File: description/ros2_control.xacro (robot description, xacro)
@@ -29,4 +29,24 @@
     </ros2_control>
     <!-- Gazebo plugin that tells Gazebo to use ros2 control -->
+    <!-- Specify UMA brand colors for Gazebo -->
+    <!-- Gazebo doesn't parse URDF colors, so we need to define them here again -->
+    <material name="gazebo_uma_blue_dark">
+        <color rgba="0 0.18 0.36 1" />
+    </material>
+    <material name="gazebo_uma_blue_light">
+        <color rgba="0.168 0.569 0.816 1" />
+    </material>
+    <material name="gazebo_uma_pink">
+        <color rgba="0.8 0 0.4 1" />
+    </material>
+    <gazebo reference='base_link'>
+        <material>Gazebo/Blue</material>
+    </gazebo>
+    <gazebo reference='link_1'>
+        <material>Gazebo/Turquoise </material>
+    </gazebo>
+    <gazebo reference='link_2'>
+        <material>Gazebo/Purple</material>
+    </gazebo>
     <gazebo>
         <plugin name="gazebo_ros2_control" filename="libgazebo_ros2_control.so">
@@ -34,3 +54,11 @@
         </plugin>
     </gazebo>
+    <gazebo>
+        <plugin name="gazebo_ros_joint_state_publisher"
+            filename="libgazebo_ros_joint_state_publisher.so">
+            <update_rate>20</update_rate>
+            <joint_name>joint_1</joint_name>
+            <joint_name>joint_2</joint_name>
+        </plugin>
+    </gazebo>
 </robot>

Commit message: update URDF to have the same joint reference frame as the control pkg

File: description/robot_core.xacro (robot description, xacro)
@@ -36,5 +36,5 @@
     <!-- - There's no upper or lower position limits -->
     <joint name="joint_1" type="continuous">
-        <origin xyz="${base_width/2 + link_1_width/2} 0 ${base_length/2}" rpy="0 0 0" />
+        <origin xyz="${base_width/2 + link_1_width/2} 0 ${base_length/2}" rpy="${-pi/2} 0 0" />
         <parent link="base_link" />
         <child link="link_1" />
