Commit message: Effort controller works

File: description/parameters.xacro (robot description, xacro)
@@ -12,4 +12,6 @@
     <xacro:property name="joint_1_velocity" value="21.9" />
     <xacro:property name="joint_1_effort" value="0.98" />
+    <xacro:property name="joint_1_min_pos" value="${-pi}" />
+    <xacro:property name="joint_1_max_pos" value="${pi}" />
     <!-- joint_2 parameters -->
     <!-- - The maximum velocity is set to 21.9 rad/s (the maximum motors velocity without load:
@@ -18,4 +20,6 @@
     <xacro:property name="joint_2_velocity" value="21.9" />
     <xacro:property name="joint_2_effort" value="0.98" />
+    <xacro:property name="joint_2_min_pos" value="${-pi}" />
+    <xacro:property name="joint_2_max_pos" value="${pi}" />
     <!-- link_1 parameters -->
     <xacro:property name="link_1_length" value="0.15" />

File: description/robot_core.xacro (robot description, xacro)
@@ -39,5 +39,5 @@
         <parent link="base_link" />
         <child link="link_1" />
-        <limit lower="0" upper="${2*pi}" velocity="${joint_1_velocity}" effort="${joint_1_effort}" />
+        <limit lower="${joint_1_min_pos}" upper="${joint_1_max_pos}" velocity="${joint_1_velocity}" effort="${joint_1_effort}" />
         <!-- <dynamics damping="1.0" friction="1.0"/> -->
     </joint>
@@ -72,5 +72,5 @@
         <parent link="link_1" />
         <child link="link_2" />
-        <limit lower="0" upper="${2*pi}" velocity="${joint_2_velocity}" effort="${joint_2_effort}" />
+        <limit lower="${joint_2_min_pos}" upper="${joint_2_max_pos}" velocity="${joint_2_velocity}" effort="${joint_2_effort}" />
         <!-- <dynamics damping="1.0" friction="1.0"/> -->
     </joint>

Commit message: improved URDF parameters

File: description/parameters.xacro (robot description, xacro)
@@ -3,6 +3,6 @@
     <!-- This file does not contain a robot description, only robot parameters -->
     <!-- base parameters-->
-    <xacro:property name="base_length" value="0.05" />
-    <xacro:property name="base_width" value="0.05" />
+    <xacro:property name="base_length" value="2" />
+    <xacro:property name="base_width" value="0.1" />
     <xacro:property name="base_mass" value="3.0" />
     <!-- joint_1 parameters -->
@@ -10,23 +10,25 @@
     210rpm) -->
     <!-- The maximum torque is set to 0.98Nm (the maximum motor torque: 10 Kg.cm) -->
-    <xacro:property name="joint_1_velocity" value="21.9" />
-    <xacro:property name="joint_1_effort" value="0.98" />
-    <xacro:property name="joint_1_min_pos" value="${-pi}" />
-    <xacro:property name="joint_1_max_pos" value="${pi}" />
+    <xacro:property name="joint_1_velocity" value="1.0" />
+    <xacro:property name="joint_1_effort" value="100" />
+    <xacro:property name="joint_1_damping" value="0.7" />
+    <!-- <xacro:property name="joint_1_min_pos" value="${-pi}" />
+    <xacro:property name="joint_1_max_pos" value="${pi}" /> -->
     <!-- joint_2 parameters -->
     <!-- - The maximum velocity is set to 21.9 rad/s (the maximum motors velocity without load:
     210rpm) -->
     <!-- The maximum torque is set to 0.98Nm (the maximum motor torque: 10 Kg.cm) -->
-    <xacro:property name="joint_2_velocity" value="21.9" />
-    <xacro:property name="joint_2_effort" value="0.98" />
-    <xacro:property name="joint_2_min_pos" value="${-pi}" />
-    <xacro:property name="joint_2_max_pos" value="${pi}" />
+    <xacro:property name="joint_2_velocity" value="1" />
+    <xacro:property name="joint_2_effort" value="100" />
+    <xacro:property name="joint_2_damping" value="0.7" />
+    <!-- <xacro:property name="joint_2_min_pos" value="${-pi}" />
+    <xacro:property name="joint_2_max_pos" value="${pi}" /> -->
     <!-- link_1 parameters -->
-    <xacro:property name="link_1_length" value="0.15" />
-    <xacro:property name="link_1_width" value="0.03" />
-    <xacro:property name="link1_mass" value="0.3" />
+    <xacro:property name="link_1_length" value="0.9" />
+    <xacro:property name="link_1_width" value="0.1" />
+    <xacro:property name="link1_mass" value="1" />
     <!-- link_2 parameters -->
-    <xacro:property name="link_2_length" value="0.15" />
-    <xacro:property name="link_2_width" value="0.03" />
-    <xacro:property name="link2_mass" value="0.3" />
+    <xacro:property name="link_2_length" value="0.9" />
+    <xacro:property name="link_2_width" value="0.1" />
+    <xacro:property name="link2_mass" value="1" />
 </robot>

File: description/robot_core.xacro (robot description, xacro)
@@ -17,5 +17,5 @@
             <origin xyz="0 0 0" rpy="0 0 0" />
             <geometry>
-                <box size="${base_width} ${base_length} ${base_length}" />
+                <box size="${base_width} ${base_width} ${base_length}" />
             </geometry>
             <material name="uma_blue_dark" />
@@ -24,10 +24,10 @@
             <origin xyz="0 0 0" rpy="0 0 0" />
             <geometry>
-                <box size="${base_width} ${base_length} ${base_length}" />
+                <box size="${base_width} ${base_width} ${base_length}" />
             </geometry>
         </collision>
-        <xacro:inertial_box mass="${base_mass}" x="${base_width}" y="${base_length}"
+        <xacro:inertial_box mass="${base_mass}" x="${base_width}" y="${base_width}"
             z="${base_length}">
-            <origin xyz="${base_width/2} ${base_length/2} ${base_length/2}" rpy="0 ${pi/2} 0" />
+            <origin xyz="${base_width/2} ${base_width/2} ${base_length/2}" rpy="0 ${pi/2} 0" />
         </xacro:inertial_box>
     </link>
@@ -35,10 +35,10 @@
     <!-- - The axis of rotation is -1 in Y, so that positive is "up" -->
     <!-- - There's no upper or lower position limits -->
-    <joint name="joint_1" type="revolute">
-        <origin xyz="${base_width/2 + link_1_width/2} 0 0" rpy="0 0 0" />
+    <joint name="joint_1" type="continuous">
+        <origin xyz="${base_width/2 + link_1_width/2} 0 ${base_length/2}" rpy="0 0 0" />
         <parent link="base_link" />
         <child link="link_1" />
-        <limit lower="${joint_1_min_pos}" upper="${joint_1_max_pos}" velocity="${joint_1_velocity}" effort="${joint_1_effort}" />
-        <!-- <dynamics damping="1.0" friction="1.0"/> -->
+        <limit velocity="${joint_1_velocity}" effort="${joint_1_effort}" />
+        <dynamics damping="${joint_1_damping}"/>
     </joint>
     <!-- link_1 describes the link_1 of the arm -->
@@ -68,10 +68,10 @@
     210rpm) -->
     <!-- The maximum torque is set to 0.98Nm (the maximum motor torque: 10 Kg.cm) -->
-    <joint name="joint_2" type="revolute">
+    <joint name="joint_2" type="continuous">
         <origin xyz="${link_1_width/2 + link_2_width/2} 0 ${link_1_length}" rpy="0 0 0" />
         <parent link="link_1" />
         <child link="link_2" />
-        <limit lower="${joint_2_min_pos}" upper="${joint_2_max_pos}" velocity="${joint_2_velocity}" effort="${joint_2_effort}" />
-        <!-- <dynamics damping="1.0" friction="1.0"/> -->
+        <limit velocity="${joint_2_velocity}" effort="${joint_2_effort}" />
+        <dynamics damping="${joint_1_damping}"/>
     </joint>
     <!-- link_2 describes the link_2 of the arm -->

Commit message: Trying to include FT sensor with errors

File: description/parameters.xacro (robot description, xacro)
@@ -12,5 +12,5 @@
     <xacro:property name="joint_1_velocity" value="1.0" />
     <xacro:property name="joint_1_effort" value="100" />
-    <xacro:property name="joint_1_damping" value="0.7" />
+    <xacro:property name="joint_1_damping" value="0.8" />
     <!-- <xacro:property name="joint_1_min_pos" value="${-pi}" />
     <xacro:property name="joint_1_max_pos" value="${pi}" /> -->
@@ -21,5 +21,5 @@
     <xacro:property name="joint_2_velocity" value="1" />
     <xacro:property name="joint_2_effort" value="100" />
-    <xacro:property name="joint_2_damping" value="0.7" />
+    <xacro:property name="joint_2_damping" value="0.8" />
     <!-- <xacro:property name="joint_2_min_pos" value="${-pi}" />
     <xacro:property name="joint_2_max_pos" value="${pi}" /> -->

File: description/ros2_control.xacro (robot description, xacro)
@@ -9,5 +9,6 @@
         <joint name="joint_1">
             <command_interface name="effort">
-                <!-- ROS uses SI units as standard, so an effort_controller connected to a rotary joint will output torque in Nm. -->
+                <!-- ROS uses SI units as standard, so an effort_controller connected to a rotary
+                joint will output torque in Nm. -->
                 <param name="min">-0.98</param>
                 <param name="max">0.98</param>
@@ -15,5 +16,5 @@
             <state_interface name="position" />
             <state_interface name="velocity" />
-            <state_interface name="effort" />
+            <!-- <state_interface name="effort" /> -->
         </joint>
         <!-- Here we include the joint_2 interface -->
@@ -25,6 +26,13 @@
             <state_interface name="position" />
             <state_interface name="velocity" />
-            <state_interface name="effort" />
+            <!-- <state_interface name="effort" /> -->
         </joint>
+        <sensor name="ee_ft_sensor">
+            <state_interface name="force.x" />
+            <state_interface name="torque.z" />
+            <param name="frame_id">EE_link</param>
+            <!-- <param name="fx_range">100</param>
+            <param name="tz_range">15</param> -->
+        </sensor>
     </ros2_control>
     <!-- Gazebo plugin that tells Gazebo to use ros2 control -->
@@ -49,4 +57,23 @@
         <material>Gazebo/Purple</material>
     </gazebo>
+    <!-- BEGIN force/torque sensor -->
+    <gazebo reference="joint_EE">
+        <provideFeedback>true</provideFeedback>
+    </gazebo>
+    <!-- The ft_sensor plugin -->
+    <gazebo>
+        <plugin filename="libgazebo_ros_ft_sensor.so" name="ee_ft_sensor">
+            <updateRate>100.0</updateRate>
+            <topicName>ft_sensor_topic</topicName>
+            <jointName>joint_EE</jointName>
+            <noise>
+                <type>gaussian</type>
+                <mean>0.0</mean>
+                <stddev>0.003</stddev>
+                <!-- change this to simulate noise -->
+            </noise>
+        </plugin>
+    </gazebo>
+    <!-- ROS 2 Control plugin -->
     <gazebo>
         <plugin name="gazebo_ros2_control" filename="libgazebo_ros2_control.so">
@@ -54,4 +81,5 @@
         </plugin>
     </gazebo>
+    <!-- Gazebo Joint State Publisher -->
     <gazebo>
         <plugin name="gazebo_ros_joint_state_publisher"
@@ -62,3 +90,12 @@
         </plugin>
     </gazebo>
+    <!-- The ft_sensor plugin -->
+    <!-- <gazebo>
+        <plugin name="ee_ft_sensor" filename="libgazebo_ros_ft_sensor.so">
+            <update_rate>200</update_rate>
+            <topicName>ee_ft_sensor/wrench</topicName>
+            <jointName>joint_EE</jointName>
+            <gaussian_noise>0.001</gaussian_noise>
+        </plugin>
+    </gazebo> -->
 </robot>

Commit message: updated arm dynamics parameters

File: description/parameters.xacro (robot description, xacro)
@@ -25,10 +25,10 @@
     <xacro:property name="joint_2_max_pos" value="${pi}" /> -->
     <!-- link_1 parameters -->
-    <xacro:property name="link_1_length" value="0.9" />
+    <xacro:property name="link_1_length" value="1.0" />
     <xacro:property name="link_1_width" value="0.1" />
-    <xacro:property name="link1_mass" value="1" />
+    <xacro:property name="link1_mass" value="3.0" />
     <!-- link_2 parameters -->
-    <xacro:property name="link_2_length" value="0.9" />
+    <xacro:property name="link_2_length" value="0.6" />
     <xacro:property name="link_2_width" value="0.1" />
-    <xacro:property name="link2_mass" value="1" />
+    <xacro:property name="link2_mass" value="2.0" />
 </robot>
